File: LM4F_BreakoutBoard/IGVC_breakout_board.sch (EAGLE design)
At the start: 4 parts

Commit message: Basic implementation almost finished. LM4F header locations added, drill holes placed, debug SMD LEDs added, phoniex connectors added.TODO: add buffer for output LED.
Parts:
- added GND_TERMINALS: MKDSN1,5/2-5,08, con-phoenix-508:MKDSN1,5/2-5,08
- added H2, H4, H5: MOUNT-HOLE3.0, holes:MOUNT-HOLE3.0
- added IC1: 7407N, 74xx-eu:7407N
- added LED1, LED2, LED3, LED4, LED5, LED6: NFSG036BT, led:NFSG036BT
- added R1, R2, R3, R4, R5, R6: (no value), resistor:R-US_M0805
Connections:
- new net GND: GND_TERMINALS-1.KL, GND_TERMINALS-2.KL, IC1P.GND, IC1P.VCC, LM4F.GND2, LM4F.VBUS, R1.1, R2.1, R3.1, R4.1, R5.1, R6.1
- new net N$10: LED3.C, R3.2
- new net N$11: LED4.C, R4.2
- new net N$12: LED5.C, R5.2
- new net N$13: LED6.C, R6.2
- new net N$14: IC1A.O, LED1.A
- new net N$15: IC1B.O, LED2.A
- new net N$16: IC1C.O, LED3.A
- new net N$17: IC1D.O, LED4.A
- new net N$18: IC1E.O, LED5.A
- new net N$19: IC1F.O, LED6.A
- new net N$20: IC1F.I, LM4F.PD0
- new net N$21: IC1E.I, LM4F.PD1
- new net N$22: IC1D.I, LM4F.PD2
- new net N$23: IC1C.I, LM4F.PD3
- new net N$24: LM4F.PD6
- new net N$25: IC1A.I, LM4F.PD7
- new net N$8: LED1.C, R1.2
- new net N$9: LED2.C, R2.2
Other:
- note added: "Debug LEDs"

Commit message: Ground plane added and traces routed. First design iteration pretty much completed and ready to test.
Parts:
- removed LED1: NFSG036BT, led:NFSG036BT
- removed R1: (no value), resistor:R-US_M0805
- added +5_CTRL: (no value), wirepad:1,6/0,8
Connections:
- removed net N$14: IC1A.O, LED1.A
- new net VBUS: IC1P.VCC, LM4F.VBUS
- net GND: no longer IC1P.VCC, LM4F.VBUS, R1.1
- net N$15: now also IC1E.O; no longer IC1B.O
- net N$16: now also IC1D.O; no longer IC1C.O
- net N$17: now also IC1C.O; no longer IC1D.O
- net N$18: now also IC1B.O; no longer IC1E.O
- net N$19: now also IC1A.O; no longer IC1F.O
- net N$20: now also IC1A.I; no longer IC1F.I
- net N$21: now also IC1B.I; no longer IC1E.I
- net N$22: now also IC1C.I; no longer IC1D.I
- net N$23: now also IC1D.I; no longer IC1C.I
- net N$24: now also IC1E.I
- net N$25: now also IC1F.I; no longer IC1A.I
- net N$8: now also +5_CTRL.P, IC1F.O; no longer LED1.C, R1.2
Other:
- moved on the sheet: IC1A, IC1B, IC1C, IC1D, IC1E, IC1F, IC1P

Commit message: Basic silk screen added to label outputs
Parts:
- renumbered LEFT_MOTOR_TERMINAL to MOTOR_TERMINALS
Changed lines of the file:
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@@
 <part name="LM4F" library="StellarisLaunchPad_Fred" deviceset="STELLARIS-LAUNCHPAD" device="STELLARIS-LAUNCHPAD-XL"/>
 <part name="FRAME1" library="frames" deviceset="A3L-LOC" device=""/>
-<part name="LEFT_MOTOR_TERMINAL" library="con-phoenix-508" deviceset="MKDSN1,5/2-5,08" device=""/>
+<part name="MOTOR_TERMINALS" library="con-phoenix-508" deviceset="MKDSN1,5/2-5,08" device=""/>
 <part name="LEFT_ENCODER_TERMINALS" library="con-phoenix-508" deviceset="MKDSN1,5/2-5,08" device=""/>
 <part name="RIGHT_ENCODER_TERMINALS" library="con-phoenix-508" deviceset="MKDSN1,5/2-5,08" device=""/>
@@
 <instance part="LM4F" gate="G$1" x="177.8" y="142.24"/>
 <instance part="FRAME1" gate="G$1" x="0" y="0"/>
-<instance part="LEFT_MOTOR_TERMINAL" gate="-1" x="134.62" y="165.1" rot="R180"/>
-<instance part="LEFT_MOTOR_TERMINAL" gate="-2" x="134.62" y="170.18" rot="R180"/>
+<instance part="MOTOR_TERMINALS" gate="-1" x="134.62" y="165.1" rot="R180"/>
+<instance part="MOTOR_TERMINALS" gate="-2" x="134.62" y="170.18" rot="R180"/>
 <instance part="LEFT_ENCODER_TERMINALS" gate="-1" x="215.9" y="175.26"/>
 <instance part="LEFT_ENCODER_TERMINALS" gate="-2" x="215.9" y="170.18"/>
@@
 <wire x1="162.56" y1="157.48" x2="152.4" y2="157.48" width="0.1524" layer="91"/>
 <wire x1="152.4" y1="157.48" x2="144.78" y2="165.1" width="0.1524" layer="91"/>
-<pinref part="LEFT_MOTOR_TERMINAL" gate="-1" pin="KL"/>
+<pinref part="MOTOR_TERMINALS" gate="-1" pin="KL"/>
 <wire x1="144.78" y1="165.1" x2="137.16" y2="165.1" width="0.1524" layer="91"/>
 <junction x="162.56" y="157.48"/>
@@
 <pinref part="LM4F" gate="G$1" pin="PA6"/>
 <wire x1="162.56" y1="160.02" x2="154.94" y2="160.02" width="0.1524" layer="91"/>
-<pinref part="LEFT_MOTOR_TERMINAL" gate="-2" pin="KL"/>
+<pinref part="MOTOR_TERMINALS" gate="-2" pin="KL"/>
 <wire x1="144.78" y1="170.18" x2="137.16" y2="170.18" width="0.1524" layer="91"/>
 <wire x1="154.94" y1="160.02" x2="144.78" y2="170.18" width="0.1524" layer="91"/>

Commit message: swapped terminals from rachel's RAS eagle lib
Parts:
- removed GND_TERMINALS, LEFT_ENCODER_TERMINALS, MOTOR_TERMINALS, RIGHT_ENCODER_TERMINALS: MKDSN1,5/2-5,08, con-phoenix-508:MKDSN1,5/2-5,08
- added GND, LEFT-ENCODER, MOTORS, RIGHT-ENCODER: PHOENIXSCREWTERMINAL_2, RASEagleLib:PHOENIXSCREWTERMINAL_2
Connections:
- net N$20 renamed LEFT
- net GND: now also GND.1, GND.2, LM4F.GND1; no longer GND_TERMINALS-1.KL, GND_TERMINALS-2.KL
- net N$1: now also RIGHT-ENCODER.2; no longer RIGHT_ENCODER_TERMINALS-2.KL
- net N$2: now also LM4F.PA6, MOTORS.2; no longer LM4F.PA7, MOTOR_TERMINALS-1.KL
- net N$3: now also LM4F.PA7, MOTORS.1; no longer LM4F.PA6, MOTOR_TERMINALS-2.KL
- net N$4: now also RIGHT-ENCODER.1; no longer RIGHT_ENCODER_TERMINALS-1.KL
- net N$5: now also LEFT-ENCODER.1; no longer LEFT_ENCODER_TERMINALS-1.KL
- net N$6: now also LEFT-ENCODER.2; no longer LEFT_ENCODER_TERMINALS-2.KL
Changed lines of the file:
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@@
 <setting verticaltext="up"/>
 </settings>
-<grid distance="0.1" unitdist="inch" unit="inch" style="dots" multiple="1" display="yes" altdistance="0.01" altunitdist="inch" altunit="inch"/>
+<grid distance="0.1" unitdist="inch" unit="inch" style="lines" multiple="1" display="no" altdistance="0.01" altunitdist="inch" altunit="inch"/>
 <layers>
 <layer number="1" name="Top" color="4" fill="1" visible="no" active="no"/>
@@
 <part name="LM4F" library="StellarisLaunchPad_Fred" deviceset="STELLARIS-LAUNCHPAD" device="STELLARIS-LAUNCHPAD-XL"/>
 <part name="FRAME1" library="frames" deviceset="A3L-LOC" device=""/>
-<part name="MOTOR_TERMINALS" library="con-phoenix-508" deviceset="MKDSN1,5/2-5,08" device=""/>
-<part name="LEFT_ENCODER_TERMINALS" library="con-phoenix-508" deviceset="MKDSN1,5/2-5,08" device=""/>
-<part name="RIGHT_ENCODER_TERMINALS" library="con-phoenix-508" deviceset="MKDSN1,5/2-5,08" device=""/>
 <part name="LED2" library="led" deviceset="NFSG036BT" device=""/>
 <part name="LED3" library="led" deviceset="NFSG036BT" device=""/>
@@
 <part name="R6" library="resistor" deviceset="R-US_" device="M0805"/>
 <part name="IC1" library="74xx-eu" deviceset="74*07" device="N"/>
-<part name="GND_TERMINALS" library="con-phoenix-508" deviceset="MKDSN1,5/2-5,08" device=""/>
 <part name="H2" library="holes" deviceset="MOUNT-HOLE" device="3.0"/>
 <part name="H4" library="holes" deviceset="MOUNT-HOLE" device="3.0"/>
 <part name="H5" library="holes" deviceset="MOUNT-HOLE" device="3.0"/>
 <part name="+5_CTRL" library="wirepad" deviceset="1,6/0,8" device=""/>
+<part name="LEFT-ENCODER" library="RASEagleLib" deviceset="PHOENIXSCREWTERMINAL_2" device=""/>
+<part name="RIGHT-ENCODER" library="RASEagleLib" deviceset="PHOENIXSCREWTERMINAL_2" device=""/>
+<part name="MOTORS" library="RASEagleLib" deviceset="PHOENIXSCREWTERMINAL_2" device=""/>
+<part name="GND" library="RASEagleLib" deviceset="PHOENIXSCREWTERMINAL_2" device=""/>
 </parts>
 <sheets>
@@
 <instance part="LM4F" gate="G$1" x="177.8" y="142.24"/>
 <instance part="FRAME1" gate="G$1" x="0" y="0"/>
-<instance part="MOTOR_TERMINALS" gate="-1" x="134.62" y="165.1" rot="R180"/>
-<instance part="MOTOR_TERMINALS" gate="-2" x="134.62" y="170.18" rot="R180"/>
-<instance part="LEFT_ENCODER_TERMINALS" gate="-1" x="215.9" y="175.26"/>
-<instance part="LEFT_ENCODER_TERMINALS" gate="-2" x="215.9" y="170.18"/>
-<instance part="RIGHT_ENCODER_TERMINALS" gate="-1" x="134.62" y="116.84" rot="R180"/>
-<instance part="RIGHT_ENCODER_TERMINALS" gate="-2" x="134.62" y="121.92" rot="R180"/>
 <instance part="LED2" gate="G$1" x="223.52" y="68.58"/>
 <instance part="LED3" gate="G$1" x="233.68" y="68.58"/>
@@
 <instance part="IC1" gate="B" x="254" y="88.9" rot="R270"/>
 <instance part="IC1" gate="A" x="264.16" y="88.9" rot="R270"/>
-<instance part="GND_TERMINALS" gate="-1" x="134.62" y="63.5" rot="R180"/>
-<instance part="GND_TERMINALS" gate="-2" x="134.62" y="68.58" rot="R180"/>
 <instance part="H2" gate="G$1" x="88.9" y="185.42"/>
 <instance part="H4" gate="G$1" x="88.9" y="53.34"/>
@@
 <instance part="+5_CTRL" gate="P" x="213.36" y="66.04" rot="R90"/>
 <instance part="IC1" gate="P" x="162.56" y="88.9"/>
+<instance part="LEFT-ENCODER" gate="G$1" x="208.28" y="172.72"/>
+<instance part="RIGHT-ENCODER" gate="G$1" x="144.78" y="116.84" rot="R180"/>
+<instance part="MOTORS" gate="G$1" x="144.78" y="157.48" rot="R180"/>
+<instance part="GND" gate="G$1" x="182.88" y="73.66" rot="R270"/>
 </instances>
 <busses>
 </busses>
 <nets>
-<net name="N$2" class="0">
-<segment>
-<pinref part="LM4F" gate="G$1" pin="PA7"/>
-<wire x1="162.56" y1="157.48" x2="152.4" y2="157.48" width="0.1524" layer="91"/>
-<wire x1="152.4" y1="157.48" x2="144.78" y2="165.1" width="0.1524" layer="91"/>
-<pinref part="MOTOR_TERMINALS" gate="-1" pin="KL"/>
-<wire x1="144.78" y1="165.1" x2="137.16" y2="165.1" width="0.1524" layer="91"/>
-<junction x="162.56" y="157.48"/>
-<junction x="137.16" y="165.1"/>
-</segment>
-</net>
-<net name="N$3" class="0">
-<segment>
-<pinref part="LM4F" gate="G$1" pin="PA6"/>
-<wire x1="162.56" y1="160.02" x2="154.94" y2="160.02" width="0.1524" layer="91"/>
-<pinref part="MOTOR_TERMINALS" gate="-2" pin="KL"/>
-<wire x1="144.78" y1="170.18" x2="137.16" y2="170.18" width="0.1524" layer="91"/>
-<wire x1="154.94" y1="160.02" x2="144.78" y2="170.18" width="0.1524" layer="91"/>
-<junction x="162.56" y="160.02"/>
-<junction x="137.16" y="170.18"/>
-</segment>
-</net>
-<net name="N$1" class="0">
-<segment>
-<pinref part="LM4F" gate="G$1" pin="PE4"/>
-<wire x1="162.56" y1="119.38" x2="147.32" y2="119.38" width="0.1524" layer="91"/>
-<wire x1="147.32" y1="119.38" x2="144.78" y2="121.92" width="0.1524" layer="91"/>
-<pinref part="RIGHT_ENCODER_TERMINALS" gate="-2" pin="KL"/>
-<wire x1="144.78" y1="121.92" x2="137.16" y2="121.92" width="0.1524" layer="91"/>
-<junction x="137.16" y="121.92"/>
-</segment>
-</net>
-<net name="N$4" class="0">
-<segment>
-<pinref part="LM4F" gate="G$1" pin="PE5"/>
-<pinref part="RIGHT_ENCODER_TERMINALS" gate="-1" pin="KL"/>
-<wire x1="162.56" y1="116.84" x2="137.16" y2="116.84" width="0.1524" layer="91"/>
-<junction x="137.16" y="116.84"/>
-</segment>
-</net>
-<net name="N$5" class="0">
-<segment>
-<pinref part="LM4F" gate="G$1" pin="PB0"/>
-<pinref part="LEFT_ENCODER_TERMINALS" gate="-1" pin="KL"/>
-<wire x1="193.04" y1="175.26" x2="213.36" y2="175.26" width="0.1524" layer="91"/>
-<junction x="193.04" y="175.26"/>
-<junction x="213.36" y="175.26"/>
-</segment>
-</net>
-<net name="N$6" class="0">
-<segment>
-<pinref part="LM4F" gate="G$1" pin="PB1"/>
-<pinref part="LEFT_ENCODER_TERMINALS" gate="-2" pin="KL"/>
-<wire x1="193.04" y1="172.72" x2="210.82" y2="172.72" width="0.1524" layer="91"/>
-<wire x1="210.82" y1="172.72" x2="213.36" y2="170.18" width="0.1524" layer="91"/>
-<junction x="193.04" y="172.72"/>
-<junction x="213.36" y="170.18"/>
-</segment>
-</net>
 <net name="N$9" class="0">
 <segment>
@@
 </segment>
 </net>
-<net name="N$20" class="0">
+<net name="LEFT" class="0">
 <segment>
 <pinref part="LM4F" gate="G$1" pin="PD0"/>
@@
 <net name="GND" class="0">
 <segment>
-<pinref part="GND_TERMINALS" gate="-2" pin="KL"/>
-<pinref part="GND_TERMINALS" gate="-1" pin="KL"/>
-<wire x1="137.16" y1="68.58" x2="137.16" y2="63.5" width="0.1524" layer="91"/>
 <pinref part="LM4F" gate="G$1" pin="GND2"/>
 <wire x1="193.04" y1="104.14" x2="193.04" y2="81.28" width="0.1524" layer="91"/>
@@
 <pinref part="R6" gate="G$1" pin="1"/>
 <wire x1="254" y1="53.34" x2="264.16" y2="53.34" width="0.1524" layer="91"/>
-<wire x1="137.16" y1="68.58" x2="193.04" y2="68.58" width="0.1524" layer="91"/>
-<junction x="193.04" y="68.58"/>
 <pinref part="IC1" gate="P" pin="GND"/>
-<wire x1="162.56" y1="81.28" x2="193.04" y2="81.28" width="0.1524" layer="91"/>
+<wire x1="162.56" y1="81.28" x2="180.34" y2="81.28" width="0.1524" layer="91"/>
 <junction x="193.04" y="81.28"/>
-<junction x="137.16" y="68.58"/>
-<junction x="137.16" y="63.5"/>
 <junction x="193.04" y="104.14"/>
 <junction x="162.56" y="81.28"/>
@@
 <junction x="254" y="53.34"/>
 <junction x="264.16" y="53.34"/>
+<pinref part="GND" gate="G$1" pin="2"/>
+<wire x1="180.34" y1="81.28" x2="185.42" y2="81.28" width="0.1524" layer="91"/>
+<wire x1="185.42" y1="81.28" x2="193.04" y2="81.28" width="0.1524" layer="91"/>
+<wire x1="180.34" y1="78.74" x2="180.34" y2="81.28" width="0.1524" layer="91"/>
+<junction x="180.34" y="81.28"/>
+<pinref part="GND" gate="G$1" pin="1"/>
+<wire x1="185.42" y1="78.74" x2="185.42" y2="81.28" width="0.1524" layer="91"/>
+<junction x="185.42" y="81.28"/>
+<pinref part="LM4F" gate="G$1" pin="GND1"/>
+<wire x1="193.04" y1="106.68" x2="193.04" y2="104.14" width="0.1524" layer="91"/>
 </segment>
 </net>
@@
 </segment>
 </net>
+<net name="N$5" class="0">
+<segment>
+<pinref part="LM4F" gate="G$1" pin="PB0"/>
+<pinref part="LEFT-ENCODER" gate="G$1" pin="1"/>
+<wire x1="193.04" y1="175.26" x2="203.2" y2="175.26" width="0.1524" layer="91"/>
+</segment>
+</net>
+<net name="N$6" class="0">
+<segment>
+<pinref part="LM4F" gate="G$1" pin="PB1"/>
+<pinref part="LEFT-ENCODER" gate="G$1" pin="2"/>
+<wire x1="193.04" y1="172.72" x2="200.66" y2="172.72" width="0.1524" layer="91"/>
+<wire x1="200.66" y1="172.72" x2="203.2" y2="170.18" width="0.1524" layer="91"/>
+</segment>
+</net>
+<net name="N$2" class="0">
+<segment>
+<pinref part="LM4F" gate="G$1" pin="PA6"/>
+<pinref part="MOTORS" gate="G$1" pin="2"/>
+<wire x1="162.56" y1="160.02" x2="149.86" y2="160.02" width="0.1524" layer="91"/>
+</segment>
+</net>
+<net name="N$3" class="0">
+<segment>
+<pinref part="LM4F" gate="G$1" pin="PA7"/>
+<pinref part="MOTORS" gate="G$1" pin="1"/>
+<wire x1="162.56" y1="157.48" x2="152.4" y2="157.48" width="0.1524" layer="91"/>
+<wire x1="152.4" y1="157.48" x2="149.86" y2="154.94" width="0.1524" layer="91"/>
+</segment>
+</net>
+<net name="N$1" class="0">
+<segment>
+<pinref part="RIGHT-ENCODER" gate="G$1" pin="2"/>
+<pinref part="LM4F" gate="G$1" pin="PE4"/>
+<wire x1="149.86" y1="119.38" x2="162.56" y2="119.38" width="0.1524" layer="91"/>
+</segment>
+</net>
+<net name="N$4" class="0">
+<segment>
+<pinref part="LM4F" gate="G$1" pin="PE5"/>
+<pinref part="RIGHT-ENCODER" gate="G$1" pin="1"/>
+<wire x1="162.56" y1="116.84" x2="152.4" y2="116.84" width="0.1524" layer="91"/>
+<wire x1="152.4" y1="116.84" x2="149.86" y2="114.3" width="0.1524" layer="91"/>
+</segment>
+</net>
